File: dolphin.kicad_sch (KiCad schematic)
At the start: 18 parts, among them J1 HRO-TYPE-C-31-M-12, J2 ISP, SW1 SW_PUSH, U1 ATMEGA32U2, U2 USBLC6-2SC6, X1 16MHz

Commit message: Add BOM/readme
Parts:
- U1: LCSC Part (none) -> C1337609; Manufacturer (none) -> Microchip Tech; Part number (none) -> ATMEGA32U2-AUR
Changed lines of the file:
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@@
+      (effects (font (size 1.27 1.27)) hide)
+    )
+    (property "LCSC Part" "C1337609" (id 4) (at 194.31 64.77 0)
+      (effects (font (size 1.27 1.27)) hide)
+    )
+    (property "Manufacturer" "Microchip Tech" (id 5) (at 194.31 64.77 0)
+      (effects (font (size 1.27 1.27)) hide)
+    )
+    (property "Part number" "ATMEGA32U2-AUR" (id 6) (at 194.31 64.77 0)
       (effects (font (size 1.27 1.27)) hide)
     )
